File: Hardware/SparkFun_Cypress_USBUART_BOB.brd (EAGLE design)
At the start: 43.2 x 20.3 mm, 29 parts, among them J3 FTDI_BASICPTH, U1 CY7C65213, U2 MIC5219 3.3V

Commit message: Ready for QC review
Parts:
- removed LOGO4: OSHW-LOGOS, SparkFun-Aesthetics:OSHW-LOGO-S
- added LOGO2: OSHW-LOGOS, SparkFun-Aesthetics:OSHW-LOGO-S
- J1: value (none) -> MICROB
Changed lines of the file:
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@@
 </element>
 <element name="FRAME1" library="SparkFun-Aesthetics" package="CREATIVE_COMMONS" value="FRAME-LETTER" x="24.13" y="-17.78"/>
-<element name="J1" library="SparkFun-Connectors" package="USB-B-MICRO-SMD_V03" value="" x="2.032" y="10.16">
+<element name="J1" library="SparkFun-Connectors" package="USB-B-MICRO-SMD_V03" value="MICROB" x="2.032" y="10.16">
 <attribute name="PROD_ID" value="CONN-11752" x="2.032" y="10.16" size="1.778" layer="27" display="off"/>
 </element>
@@
 <element name="FD1" library="SparkFun-Aesthetics" package="MICRO-FIDUCIAL" value="FIDUCIALUFIDUCIAL" x="5.08" y="1.27"/>
 <element name="FD2" library="SparkFun-Aesthetics" package="MICRO-FIDUCIAL" value="FIDUCIALUFIDUCIAL" x="39.37" y="19.05"/>
-<element name="LOGO4" library="SparkFun-Aesthetics" package="OSHW-LOGO-S" value="OSHW-LOGOS" x="2.54" y="1.905" rot="MR0"/>
 <element name="LOGO5" library="SparkFun-Aesthetics" package="SFE_LOGO_FLAME_.2" value="SFE_LOGO_FLAME.2_INCH" x="6.223" y="10.287"/>
 <element name="D4" library="SparkFun-DiscreteSemi" package="SOD-323" value="5.6V" x="7.62" y="6.35" rot="R180">
@@
 <attribute name="PROD_ID" value="CAP-10300" x="3.175" y="7.62" size="0.8128" layer="27" font="vector" ratio="15" rot="R180" display="off"/>
 </element>
+<element name="LOGO2" library="SparkFun-Aesthetics" package="OSHW-LOGO-S" value="OSHW-LOGOS" x="2.794" y="1.905" rot="MR0"/>
 </elements>
 <signals>
@@
 <wire x1="13.97" y1="19.05" x2="13.97" y2="17.907" width="0.8128" layer="16"/>
 <wire x1="13.97" y1="17.907" x2="13.589" y2="17.526" width="0.8128" layer="16"/>
-<wire x1="13.589" y1="17.526" x2="5.588" y2="17.526" width="0.8128" layer="16"/>
-<wire x1="5.588" y1="17.526" x2="5.334" y2="17.272" width="0.8128" layer="16"/>
-<wire x1="5.334" y1="17.272" x2="5.334" y2="3.302" width="0.8128" layer="16"/>
+<wire x1="13.589" y1="17.526" x2="5.715" y2="17.526" width="0.8128" layer="16"/>
+<wire x1="5.715" y1="17.526" x2="5.334" y2="17.145" width="0.8128" layer="16"/>
+<wire x1="5.334" y1="17.145" x2="5.334" y2="3.302" width="0.8128" layer="16"/>
 <via x="5.969" y="2.794" extent="1-16" drill="0.381"/>
 <wire x1="5.969" y1="2.794" x2="13.97" y2="2.794" width="0.8128" layer="1"/>
