File: Hardware/SparkFun_Cypress_USBUART_BOB.brd (EAGLE design)
At the start: 43.2 x 20.3 mm, 31 parts, among them J1 MICROB, J3 FTDI_BASICPTH, U1 CY7C65213, U2 3.3V

Commit message: Update to v10, ready for reds
Other:
- board text added: "v10"
- board text removed: "v04"
Changed lines of the file:
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@@
 <?xml version="1.0" encoding="utf-8"?>
 <!DOCTYPE eagle SYSTEM "eagle.dtd">
-<eagle version="7.6.0">
+<eagle version="7.5.0">
 <drawing>
 <settings>
@@
 <layer number="20" name="Dimension" color="15" fill="1" visible="yes" active="yes"/>
 <layer number="21" name="tPlace" color="16" fill="1" visible="yes" active="yes"/>
-<layer number="22" name="bPlace" color="14" fill="1" visible="no" active="yes"/>
+<layer number="22" name="bPlace" color="14" fill="1" visible="yes" active="yes"/>
 <layer number="23" name="tOrigins" color="15" fill="1" visible="yes" active="yes"/>
-<layer number="24" name="bOrigins" color="15" fill="1" visible="no" active="yes"/>
-<layer number="25" name="tNames" color="7" fill="1" visible="yes" active="yes"/>
+<layer number="24" name="bOrigins" color="15" fill="1" visible="yes" active="yes"/>
+<layer number="25" name="tNames" color="7" fill="1" visible="no" active="yes"/>
 <layer number="26" name="bNames" color="7" fill="1" visible="no" active="yes"/>
 <layer number="27" name="tValues" color="7" fill="1" visible="no" active="yes"/>
@@
 <layer number="43" name="vRestrict" color="2" fill="10" visible="no" active="yes"/>
 <layer number="44" name="Drills" color="7" fill="1" visible="no" active="yes"/>
-<layer number="45" name="Holes" color="7" fill="1" visible="no" active="yes"/>
+<layer number="45" name="Holes" color="7" fill="1" visible="yes" active="yes"/>
 <layer number="46" name="Milling" color="3" fill="1" visible="no" active="yes"/>
 <layer number="47" name="Measures" color="7" fill="1" visible="no" active="yes"/>
-<layer number="51" name="tDocu" color="6" fill="1" visible="no" active="yes"/>
+<layer number="51" name="tDocu" color="6" fill="1" visible="yes" active="yes"/>
 <layer number="52" name="bDocu" color="7" fill="1" visible="no" active="yes"/>
 <layer number="3" name="Route3" color="4" fill="3" visible="no" active="no"/>
@@
 <text x="0.635" y="18.542" size="0.8128" layer="22" font="vector" ratio="15" rot="MR180" align="center-left">CY7C65213
 USBUART</text>
-<text x="2.54" y="16.51" size="0.8128" layer="16" font="vector" ratio="15" rot="MR0" align="center-left">v04</text>
+<text x="2.54" y="16.51" size="0.8128" layer="16" font="vector" ratio="15" rot="MR0" align="center-left">v10</text>
 <text x="54.61" y="-17.78" size="1.778" layer="51" font="vector" ratio="10">Mike Hord</text>
 <dimension x1="0" y1="20.32" x2="0" y2="0" x3="-7.62" y3="10.16" textsize="1.778" textratio="10" layer="47" dtype="vertical" width="0.254" unit="inch"/>
