File: Hardware/SparkFun_Cypress_USBUART_BOB.sch (EAGLE design)
At the start: 31 parts, among them J1 MICROB, J3 FTDI_BASICPTH, U1 CY7C65213, U2 3.3V

Commit message: Remove 15-ohm resistor in power line
Parts:
- removed R2: 15, SparkFun-Resistors:15OHM-1/10W-1%(0603)0603
Connections:
- removed net 5V_CLAMPED: C3.1, C4.1, D4.C, JP1.3, R2.2, U1.VCC
- net 5V: now also C3.1, C4.1, D4.C, JP1.3, U1.VCC; no longer R2.1
Changed lines of the file:
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@@
 <?xml version="1.0" encoding="utf-8"?>
 <!DOCTYPE eagle SYSTEM "eagle.dtd">
-<eagle version="7.5.0">
+<eagle version="7.6.0">
 <drawing>
 <settings>
@@
 <layer number="255" name="routoute" color="7" fill="1" visible="yes" active="yes"/>
 </layers>
-<schematic xreflabel="%F%N/%S" xrefpart="/%S.%C%R">
+<schematic xreflabel="%F%N/%S" xrefpart="1_/%S.%C%R">
 <attributes>
 </attributes>
@@
 <part name="C2" library="SparkFun-Capacitors" deviceset="1.0UF-16V-10%(0603)" device="" value="1.0uF"/>
 <part name="SUPPLY3" library="SparkFun-Aesthetics" deviceset="VDD" device=""/>
-<part name="5V_CLAMPED" library="SparkFun-Aesthetics" deviceset="5V" device="" value="5V_CLAMPED"/>
 <part name="SUPPLY5" library="SparkFun-Aesthetics" deviceset="VCCIO" device=""/>
 <part name="SUPPLY6" library="SparkFun-Aesthetics" deviceset="VDD" device=""/>
@@
 <part name="GND4" library="SparkFun-Aesthetics" deviceset="GND" device=""/>
 <part name="SUPPLY10" library="SparkFun-Aesthetics" deviceset="VCCIO" device=""/>
-<part name="SUPPLY12" library="SparkFun-Aesthetics" deviceset="5V" device="" value="5V_CLAMPED"/>
 <part name="SUPPLY13" library="SparkFun-Aesthetics" deviceset="3.3V" device=""/>
 <part name="JP2" library="SparkFun-Passives" deviceset="JUMPER-PAD-2-NO" device="YES_SILK"/>
@@
 <part name="FD2" library="SparkFun-Aesthetics" deviceset="FIDUCIAL" device="UFIDUCIAL"/>
 <part name="D4" library="SparkFun-DiscreteSemi" deviceset="DIODE-ZENER" device="5.6V" value="5.6V"/>
-<part name="R2" library="SparkFun-Resistors" deviceset="15OHM-1/10W-1%(0603)" device="0603" value="15"/>
 <part name="SUPPLY4" library="SparkFun-Aesthetics" deviceset="5V" device=""/>
-<part name="5V_CLAMPED1" library="SparkFun-Aesthetics" deviceset="5V" device="" value="5V_CLAMPED"/>
 <part name="GND8" library="SparkFun-Aesthetics" deviceset="GND" device=""/>
 <part name="C3" library="SparkFun-Capacitors" deviceset="0.1UF-25V-5%(0603)" device="" value="0.1uF"/>
 <part name="C4" library="SparkFun-Capacitors" deviceset="4.7UF-16V-20%,+80%-(1206)" device="" value="4.7uF"/>
-<part name="SUPPLY9" library="SparkFun-Aesthetics" deviceset="5V" device="" value="5V_CLAMPED"/>
 <part name="C5" library="SparkFun-Capacitors" deviceset="0.1UF-25V-5%(0603)" device="" value="0.1uF"/>
 <part name="C6" library="SparkFun-Capacitors" deviceset="4.7UF-16V-20%,+80%-(1206)" device="" value="4.7uF"/>
@@
 <part name="C8" library="SparkFun-Capacitors" deviceset="10PF-50V-5%(0603)" device="" value="10pF"/>
 <part name="SUPPLY21" library="SparkFun-Aesthetics" deviceset="VCCIO" device=""/>
+<part name="SUPPLY9" library="SparkFun-Aesthetics" deviceset="5V" device=""/>
+<part name="SUPPLY12" library="SparkFun-Aesthetics" deviceset="5V" device=""/>
+<part name="SUPPLY24" library="SparkFun-Aesthetics" deviceset="5V" device=""/>
 </parts>
 <sheets>
@@
 <instance part="C2" gate="G$1" x="7.62" y="147.32"/>
 <instance part="SUPPLY3" gate="VDD" x="101.6" y="172.72"/>
-<instance part="5V_CLAMPED" gate="G$1" x="99.06" y="175.26"/>
 <instance part="SUPPLY5" gate="G$1" x="104.14" y="170.18"/>
 <instance part="SUPPLY6" gate="VDD" x="7.62" y="160.02"/>
@@
 <instance part="GND4" gate="1" x="22.86" y="63.5"/>
 <instance part="SUPPLY10" gate="G$1" x="33.02" y="109.22"/>
-<instance part="SUPPLY12" gate="G$1" x="17.78" y="116.84"/>
 <instance part="SUPPLY13" gate="G$1" x="25.4" y="114.3"/>
 <instance part="JP2" gate="G$1" x="40.64" y="106.68" smashed="yes">
@@
 <instance part="FD2" gate="G$1" x="243.84" y="25.4"/>
 <instance part="D4" gate="G$1" x="43.18" y="35.56" rot="R90"/>
-<instance part="R2" gate="G$1" x="33.02" y="43.18"/>
-<instance part="SUPPLY4" gate="G$1" x="20.32" y="45.72"/>
-<instance part="5V_CLAMPED1" gate="G$1" x="43.18" y="45.72"/>
+<instance part="SUPPLY4" gate="G$1" x="43.18" y="45.72"/>
 <instance part="GND8" gate="1" x="43.18" y="27.94"/>
 <instance part="C3" gate="G$1" x="30.48" y="147.32"/>
 <instance part="C4" gate="G$1" x="40.64" y="147.32"/>
-<instance part="SUPPLY9" gate="G$1" x="30.48" y="160.02"/>
 <instance part="C5" gate="G$1" x="50.8" y="147.32"/>
 <instance part="C6" gate="G$1" x="60.96" y="147.32"/>
@@
 </instance>
 <instance part="SUPPLY21" gate="G$1" x="228.6" y="165.1"/>
+<instance part="SUPPLY9" gate="G$1" x="99.06" y="175.26"/>
+<instance part="SUPPLY12" gate="G$1" x="30.48" y="160.02"/>
+<instance part="SUPPLY24" gate="G$1" x="17.78" y="116.84"/>
 </instances>
 <busses>
@@
 </segment>
 <segment>
+<wire x1="116.84" y1="160.02" x2="99.06" y2="160.02" width="0.1524" layer="91"/>
+<wire x1="99.06" y1="160.02" x2="99.06" y2="175.26" width="0.1524" layer="91"/>
+<pinref part="U1" gate="G$1" pin="VCC"/>
+<pinref part="SUPPLY9" gate="G$1" pin="5V"/>
+</segment>
+<segment>
+<pinref part="C3" gate="G$1" pin="1"/>
+<wire x1="30.48" y1="160.02" x2="30.48" y2="157.48" width="0.1524" layer="91"/>
+<pinref part="C4" gate="G$1" pin="1"/>
+<wire x1="30.48" y1="157.48" x2="30.48" y2="152.4" width="0.1524" layer="91"/>
+<wire x1="30.48" y1="157.48" x2="40.64" y2="157.48" width="0.1524" layer="91"/>
+<wire x1="40.64" y1="157.48" x2="40.64" y2="152.4" width="0.1524" layer="91"/>
+<junction x="30.48" y="157.48"/>
+<pinref part="SUPPLY12" gate="G$1" pin="5V"/>
+</segment>
+<segment>
+<wire x1="17.78" y1="116.84" x2="17.78" y2="99.06" width="0.1524" layer="91"/>
+<pinref part="JP1" gate="G$1" pin="3"/>
+<wire x1="17.78" y1="99.06" x2="25.4" y2="99.06" width="0.1524" layer="91"/>
+<wire x1="25.4" y1="99.06" x2="25.4" y2="101.6" width="0.1524" layer="91"/>
+<pinref part="SUPPLY24" gate="G$1" pin="5V"/>
+</segment>
+<segment>
+<pinref part="D4" gate="G$1" pin="C"/>
+<wire x1="43.18" y1="38.1" x2="43.18" y2="45.72" width="0.1524" layer="91" style="longdash"/>
 <pinref part="SUPPLY4" gate="G$1" pin="5V"/>
-<wire x1="20.32" y1="45.72" x2="20.32" y2="43.18" width="0.1524" layer="91" style="longdash"/>
-<pinref part="R2" gate="G$1" pin="1"/>
-<wire x1="20.32" y1="43.18" x2="27.94" y2="43.18" width="0.1524" layer="91" style="longdash"/>
 </segment>
 </net>
@@
 </segment>
 </net>
-<net name="5V_CLAMPED" class="0">
-<segment>
-<pinref part="5V_CLAMPED" gate="G$1" pin="5V"/>
-<wire x1="116.84" y1="160.02" x2="99.06" y2="160.02" width="0.1524" layer="91"/>
-<wire x1="99.06" y1="160.02" x2="99.06" y2="175.26" width="0.1524" layer="91"/>
-<pinref part="U1" gate="G$1" pin="VCC"/>
-</segment>
-<segment>
-<pinref part="D4" gate="G$1" pin="C"/>
-<wire x1="43.18" y1="38.1" x2="43.18" y2="43.18" width="0.1524" layer="91" style="longdash"/>
-<pinref part="R2" gate="G$1" pin="2"/>
-<wire x1="43.18" y1="43.18" x2="38.1" y2="43.18" width="0.1524" layer="91" style="longdash"/>
-<pinref part="5V_CLAMPED1" gate="G$1" pin="5V"/>
-<wire x1="43.18" y1="45.72" x2="43.18" y2="43.18" width="0.1524" layer="91" style="longdash"/>
-<junction x="43.18" y="43.18"/>
-</segment>
-<segment>
-<pinref part="SUPPLY12" gate="G$1" pin="5V"/>
-<wire x1="17.78" y1="116.84" x2="17.78" y2="99.06" width="0.1524" layer="91"/>
-<pinref part="JP1" gate="G$1" pin="3"/>
-<wire x1="17.78" y1="99.06" x2="25.4" y2="99.06" width="0.1524" layer="91"/>
-<wire x1="25.4" y1="99.06" x2="25.4" y2="101.6" width="0.1524" layer="91"/>
-</segment>
-<segment>
-<pinref part="SUPPLY9" gate="G$1" pin="5V"/>
-<pinref part="C3" gate="G$1" pin="1"/>
-<wire x1="30.48" y1="160.02" x2="30.48" y2="157.48" width="0.1524" layer="91"/>
-<pinref part="C4" gate="G$1" pin="1"/>
-<wire x1="30.48" y1="157.48" x2="30.48" y2="152.4" width="0.1524" layer="91"/>
-<wire x1="30.48" y1="157.48" x2="40.64" y2="157.48" width="0.1524" layer="91"/>
-<wire x1="40.64" y1="157.48" x2="40.64" y2="152.4" width="0.1524" layer="91"/>
-<junction x="30.48" y="157.48"/>
-</segment>
-</net>

Commit message: Update to v10, ready for reds
Other:
- note added: "10"
- note removed: "04"
Changed lines of the file:
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@@
 <?xml version="1.0" encoding="utf-8"?>
 <!DOCTYPE eagle SYSTEM "eagle.dtd">
-<eagle version="7.6.0">
+<eagle version="7.5.0">
 <drawing>
 <settings>
@@
 <layer number="255" name="routoute" color="7" fill="1" visible="yes" active="yes"/>
 </layers>
-<schematic xreflabel="%F%N/%S" xrefpart="1_/%S.%C%R">
+<schematic xreflabel="%F%N/%S" xrefpart="/%S.%C%R">
 <attributes>
 </attributes>
@@
 <sheet>
 <plain>
-<text x="237.998" y="6.35" size="3.81" layer="94" font="vector">04</text>
+<text x="237.998" y="6.35" size="3.81" layer="94" font="vector">10</text>
 <text x="154.432" y="6.096" size="3.81" layer="94" font="vector">Mike Hord</text>
 <text x="27.94" y="95.25" size="1.27" layer="97" font="vector">Open JP1 if VIO used
